Commit message: adv_lecture: add dynamic, sim, orientation
x#	new file:   adv_lecture/cfg/sample1.cfg

File: sim_lecture/urdf/simple_robot1.urdf (robot description, URDF)
Before this commit: robot my_robo, 2 links, 1 joints
Links:
- removed link my_link
- added link body_link, mass 1; collision box size=1 1 1; visual box size=1 1 1
Joints:
- joint joint1: child my_link -> body_link
