Commit message: sim_lecture: add

File: sim_lecture/urdf/wheel_robot3.urdf (robot description, URDF)
Before this commit: robot my_robo, 6 links, 5 joints
Links:
- link body_link: mass 1.0 -> 2.0
- link left_wheel_link: mass 0.3 -> 0.1
- link right_wheel_link: mass 0.3 -> 0.1
Joints:
- joint left_wheel_joint: limit (none) -> effort=0.4 velocity=12.0
- joint right_wheel_joint: limit (none) -> effort=0.4 velocity=12.0; origin xyz=0 -0.1 0.05 rpy=1.5708 0 0 -> xyz=0 -0.1 0.05 rpy=-1.5708 0 0
