Commit message: sim_lecture: add lecture# Please enter the commit message for your changes. Lines starting

File: sim_lecture/urdf/wheel_robot6.urdf (robot description, URDF)
Before this commit: robot my_robo, 7 links, 6 joints
Links:
- removed link base_footprint
- removed link rear_ball_link
- added link front_steer_link, mass 0.1; visual cylinder length=0.04 radius=0.01
- added link front_wheel_link, mass 0.3; collision cylinder length=0.02 radius=0.015; visual cylinder length=0.02 radius=0.015
- added link imu_link
Joints:
- removed joint base_joint
- removed joint body_joint
- removed joint rear_ball_joint
- added joint bodyjoint: type fixed, parent base_link, child body_link, origin xyz=0.05 0 0.07 rpy=0 0 0
- added joint front_steer_joint: type continuous, parent base_link, child front_steer_link, origin xyz=0.14 0 0.05 rpy=0 0 0, axis 0 0 1
- added joint front_wheel_joint: type continuous, parent front_steer_link, child front_wheel_link, origin xyz=-0.01 0 -0.035 rpy=1.5708 0 0, axis 0 0 1
- added joint imu_joint: type fixed, parent body_link, child imu_link, origin xyz=0 0 0 rpy=0 0 0
- joint left_wheel_joint: limit effort=0.7 velocity=20.0 -> effort=0.4 velocity=12.0
- joint lidar_joint: origin xyz=0.09 0 0.05 rpy=0 0 0 -> xyz=0.10 0 0.05 rpy=0 0 0
- joint right_wheel_joint: limit effort=0.7 velocity=20.0 -> effort=0.4 velocity=12.0
