Commit message: nav_lecture: add lecture

File: nav_lecture/urdf/wheel_robot_normal.urdf (robot description, URDF)
Before this commit: robot my_robo, 7 links, 6 joints
Links:
- removed link base_footprint
- removed link base_link
- removed link body_link
- removed link left_wheel_link
- removed link lidar_link
- removed link rear_ball_link
- removed link right_wheel_link
- added link /wheel_robot/base_link
- added link /wheel_robot/body_link, mass 2.0; collision box size=0.23 0.18 0.05; visual box size=0.24 0.19 0.06
- added link /wheel_robot/left_wheel_link, mass 0.1; collision cylinder length=0.01 radius=0.05; visual cylinder length=0.01 radius=0.05
- added link /wheel_robot/lidar_link; collision cylinder length=0.06 radius=0.02; visual cylinder length=0.06 radius=0.02
- added link /wheel_robot/rear_ball_link, mass 0.1; collision sphere radius=0.04; visual sphere radius=0.04
- added link /wheel_robot/right_wheel_link, mass 0.1; collision cylinder length=0.01 radius=0.05; visual cylinder length=0.01 radius=0.05
Joints:
- removed joint base_joint
- removed joint body_joint
- removed joint left_wheel_joint
- removed joint lidar_joint
- removed joint rear_ball_joint
- removed joint right_wheel_joint
- added joint /wheel_robot/body_joint: type fixed, parent /wheel_robot/base_link, child /wheel_robot/body_link, origin xyz=-0.08 0 0.07 rpy=0 0 0
- added joint /wheel_robot/left_wheel_joint: type continuous, parent /wheel_robot/base_link, child /wheel_robot/left_wheel_link, origin xyz=0 0.1 0.05 rpy=-1.5708 0 0, axis 0 0 1, limit effort=0.7 velocity=20.0
- added joint /wheel_robot/lidar_joint: type fixed, parent /wheel_robot/body_link, child /wheel_robot/lidar_link, origin xyz=0.09 0 0.05 rpy=0 0 0
- added joint /wheel_robot/rear_ball_joint: type fixed, parent /wheel_robot/base_link, child /wheel_robot/rear_ball_link, origin xyz=-0.15 0 0.04 rpy=0 0 0, axis 0 0 1
- added joint /wheel_robot/right_wheel_joint: type continuous, parent /wheel_robot/base_link, child /wheel_robot/right_wheel_link, origin xyz=0 -0.1 0.05 rpy=-1.5708 0 0, axis 0 0 1, limit effort=0.7 velocity=20.0

Commit message: nav_lecture: modify robot config

File: nav_lecture/urdf/wheel_robot_normal.urdf (robot description, URDF)
Before this commit: robot my_robo, 6 links, 5 joints
Links:
- link /wheel_robot/left_wheel_link: mass 0.1 -> 0.03
- link /wheel_robot/right_wheel_link: mass 0.1 -> 0.03
